File: UnwaryNuc.sch (KiCad schematic (older format))
At the start: 30 parts, among them Q1 2N3904, U1 NUC980DF71YC, U2 LAN8740A-EN-TR, U3 LAN8740A-EN-TR, U4 LD3985G18R_TSOT23, U5 LDK130-33_SOT23_SOT353

Commit message: added supply sequencing and stuff
Parts:
- removed U5: LDK130-33_SOT23_SOT353, Package_TO_SOT_SMD:SOT-23-5_HandSoldering, symbol Regulator_Linear:LDK130-33_SOT23_SOT353
- added C22, C3: 8pf, Capacitor_SMD:C_0603_1608Metric_Pad1.05x0.95mm_HandSolder, symbol Device:C
- added C23, C24: 7pf, Capacitor_SMD:C_0603_1608Metric_Pad1.05x0.95mm_HandSolder, symbol Device:C
- added C25: T491D226k035AT, Capacitor_Tantalum_SMD:CP_EIA-7343-15_Kemet-W_Pad2.25x2.55mm_HandSolder, symbol Device:C
- added C26: 293D127X96, Capacitor_Tantalum_SMD:CP_EIA-7343-43_Kemet-X_Pad2.25x2.55mm_HandSolder, symbol Device:C
- added C27, C29, C30, C31, C32, C? (x2): 1u, Capacitor_SMD:C_1206_3216Metric_Pad1.42x1.75mm_HandSolder, symbol Device:C
- added C28: 10n, Capacitor_SMD:C_1206_3216Metric_Pad1.42x1.75mm_HandSolder, symbol Device:C
- added D3: B240, 40V 2A, Diode_SMD:D_SMB_Handsoldering, symbol Diode:B240
- added L1: CDRH6D38NP-150NC, UnwaryNuc:CDRH6D38_Sumida, symbol Device:L
- added Q? (x2): BC856BDW1, Package_TO_SOT_SMD:SOT-363_SC-70-6, symbol Transistor_BJT:BC856BDW1
- added R2, R3, R? (x4): 100k, Resistor_SMD:R_0805_2012Metric_Pad1.15x1.40mm_HandSolder, symbol Device:R
- added R4: 3.01k, Resistor_SMD:R_0805_2012Metric_Pad1.15x1.40mm_HandSolder, symbol Device:R
- added R5: 1.78k, Resistor_SMD:R_0805_2012Metric_Pad1.15x1.40mm_HandSolder, symbol Device:R
- added U5: MIC4690, Package_SO:SOIC-8_3.9x4.9mm_P1.27mm, symbol Regulator_Switching:MIC4690
- added U?: LM3880, Package_TO_SOT_SMD:SOT-23-6, symbol Power_Supervisor:LM3880
- added U?: AP2127K-1.2, Package_TO_SOT_SMD:SOT-23-5, symbol Regulator_Linear:AP2127K-1.2
- added Y1: ABS07-166, Crystal:Crystal_SMD_3215-2Pin_3.2x1.5mm, symbol Device:Crystal
- added Y2: NX5032GA, Crystal:Crystal_SMD_5032-2Pin_5.0x3.2mm_HandSoldering, symbol Device:Crystal
- U4: value LD3985G18R_TSOT23 -> LD3985M18R_TSOT23
Connections:
- net labels added: 1V2EN, 1V8_EN, 3V3EN, nRST
- wire segments 89 -> 169
- no-connect marks 0 -> 1
Other:
- moved on the sheet: BT1, C1, D1, D2, U4

Commit message: usb's connected, rmii nets assigned, some placement done
Parts:
- added C35, C36, C37: 1u, Capacitor_SMD:C_1206_3216Metric_Pad1.42x1.75mm_HandSolder, symbol Device:C
- added D4: D, Diode_SMD:D_SOD-523, symbol Device:D
- added FB1: Ferrite_Bead_Small, Inductor_SMD:L_1206_3216Metric_Pad1.42x1.75mm_HandSolder, symbol Device:Ferrite_Bead_Small
- added J1: USB_B_Micro, Connector_USB:USB_Micro-B_Molex_47346-0001, symbol Connector:USB_B_Micro
- added J2: USB_A_Dual, Connector_USB:USB_A_Wuerth_61400826021_Horizontal_Stacked, symbol Connector_Unwary:USB_A_Dual
- added J3: Conn_01x06_Male, Connector_PinHeader_2.54mm:PinHeader_1x06_P2.54mm_Vertical, symbol Connector:Conn_01x06_Male
- added J4, J5: RJ45_Amphenol_RJMG1BD3B8K1ANR, Connector_RJ:RJ45_Amphenol_RJMG1BD3B8K1ANR, symbol Connector:RJ45_Amphenol_RJMG1BD3B8K1ANR
- added R10: 100k, Resistor_SMD:R_0805_2012Metric_Pad1.15x1.40mm_HandSolder, symbol Device:R
- added R11, R12: 27, Resistor_SMD:R_0603_1608Metric_Pad1.05x0.95mm_HandSolder, symbol Device:R
- added R13, R14: R, Resistor_SMD:R_0603_1608Metric_Pad1.05x0.95mm_HandSolder, symbol Device:R
- added R15, R16: 12.1k, Resistor_SMD:R_0603_1608Metric_Pad1.05x0.95mm_HandSolder, symbol Device:R
- added R17, R18, R19, R20: 4.7, Resistor_SMD:R_0603_1608Metric_Pad1.05x0.95mm_HandSolder, symbol Device:R
- added SW1: SW_SPST, Button_Switch_SMD:SW_SPST_CK_RS282G05A3, symbol Switch:SW_SPST
- added TP1, TP2: TestPoint, TestPoint:TestPoint_Keystone_5019_Minature, symbol Connector:TestPoint
- BT1: footprint (none) -> Battery:Battery_Panasonic_CR2032-VS1N_Vertical_CircularHoles
- D1, D2: footprint (none) -> Diode_SMD:D_SOD-523
- gave numbers to parts that had none: 9
Connections:
- net labels added: +5V, RMII0_CRSDV, RMII0_MDC, RMII0_MDIO, RMII0_REFCLK, RMII0_RXD0, RMII0_RXD1, RMII0_RXERR, RMII0_TXD0, RMII0_TXD1, RMII0_TXEN, RMII1_CRSDV, RMII1_MDC, RMII1_MDIO, RMII1_REFCLK, RMII1_RXD0, RMII1_RXD1, RMII1_RXERR, RMII1_TXD0, RMII1_TXD1, RMII1_TXEN, UART0_RXD, UART0_TXD, USB0.DD_N, USB0.DD_P, USB0_VBUSVLD, USBHL.DD_N, USBHL.DD_P, VBUS
- wire segments 169 -> 268
Other:
- note added: "Reset"
- note added: "Supplies and Sequencing\n"
- moved on the sheet: BT1, C1, C2, C25, C26, C27, C28, C29, C33, C34, D1, D2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
