File: UnwaryNuc.kicad_pcb (KiCad board)
At the start: 4 copper layers, 106.1 x 63.5 mm, 117 parts, among them J1 USB_B_Micro, J2 USB_A_Dual, J3 Conn_01x06_Male, J4 RJ45_Amphenol_RJMG1BD3B8K1ANR, J5 RJ45_Amphenol_RJMG1BD3B8K1ANR, Q1 2N3904, Q2 BC856BDW1, SW1 SW_SPST, U1 NUC980DF71YC, U2 LAN8740A-EN-TR, U3 LAN8740A-EN-TR, U4 LD3985M18R_TSOT23, U5 MIC4690, U6 LM3880, U7 AP2127K-1.2, Y1 ABS07-166, Y2 NX5032GA

Commit message: pushing up to pull to desktop
Parts:
- moved R23 66.2 mm to (144.6, 73.8), turned to 90 degrees
- moved R25 63.1 mm to (141.2, 73.8), turned to 90 degrees
- moved R24 62.8 mm to (142.8, 73.8), turned to 90 degrees
- moved R22 43.3 mm to (146.2, 73.8), turned to 90 degrees
- moved R21 41.7 mm to (147.9, 73.8), turned to 90 degrees
Changed lines of the file:
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@@
   )
   (module Resistor_SMD:R_0603_1608Metric_Pad1.05x0.95mm_HandSolder (layer "L1_(Top)")
-    (at 93.7 32.26)
+    (at 141.15 73.8 90)
     (descr "Resistor SMD 0603 (1608 Metric), square (rectangular) end terminal, IPC_7351 nominal with elongated pad for handsoldering. (Body size source: http://www.tortai-tech.com/upload/download/2011102023233369053.pdf), generated with kicad-footprint-generator")
     (tags "resistor handsolder")
     (attr smd)
-    (fp_text reference R25 (at 0 -1.43) (layer F.SilkS)
+    (fp_text reference R25 (at 0 -1.43 90) (layer F.SilkS)
       (effects (font (size 1 1) (thickness 0.15)))
     )
-    (fp_text value 100 (at 0 1.43) (layer F.Fab)
+    (fp_text value 100 (at 0 1.43 90) (layer F.Fab)
       (effects (font (size 1 1) (thickness 0.15)))
     )
-    (fp_text user %R (at 0 0) (layer F.Fab)
+    (fp_text user %R (at 0 0 90) (layer F.Fab)
       (effects (font (size 0.4 0.4) (thickness 0.06)))
     )
@@
     (fp_line (start -0.8 -0.4) (end 0.8 -0.4) (layer F.Fab) (width 0.1))
     (fp_line (start -0.8 0.4) (end -0.8 -0.4) (layer F.Fab) (width 0.1))
-    (pad 2 smd roundrect (at 0.875 0) (size 1.05 0.95) (layers "L1_(Top)" F.Paste F.Mask) (roundrect_rratio 0.25)
+    (pad 2 smd roundrect (at 0.875 0 90) (size 1.05 0.95) (layers "L1_(Top)" F.Paste F.Mask) (roundrect_rratio 0.25)
       (net 244 "Net-(R25-Pad2)"))
-    (pad 1 smd roundrect (at -0.875 0) (size 1.05 0.95) (layers "L1_(Top)" F.Paste F.Mask) (roundrect_rratio 0.25)
+    (pad 1 smd roundrect (at -0.875 0 90) (size 1.05 0.95) (layers "L1_(Top)" F.Paste F.Mask) (roundrect_rratio 0.25)
       (net 225 /RMII0_REFCLK))
     (model ${KISYS3DMOD}/Resistor_SMD.3dshapes/R_0603_1608Metric.wrl
@@
   )
   (module Resistor_SMD:R_0603_1608Metric_Pad1.05x0.95mm_HandSolder (layer "L1_(Top)")
-    (at 98.05 29.75)
+    (at 142.85 73.8 90)
     (descr "Resistor SMD 0603 (1608 Metric), square (rectangular) end terminal, IPC_7351 nominal with elongated pad for handsoldering. (Body size source: http://www.tortai-tech.com/upload/download/2011102023233369053.pdf), generated with kicad-footprint-generator")
     (tags "resistor handsolder")
     (attr smd)
-    (fp_text reference R24 (at 0 -1.43) (layer F.SilkS)
+    (fp_text reference R24 (at 0 -1.43 90) (layer F.SilkS)
       (effects (font (size 1 1) (thickness 0.15)))
     )
-    (fp_text value 100 (at 0 1.43) (layer F.Fab)
+    (fp_text value 100 (at 0 1.43 90) (layer F.Fab)
       (effects (font (size 1 1) (thickness 0.15)))
     )
-    (fp_text user %R (at 0 0) (layer F.Fab)
+    (fp_text user %R (at 0 0 90) (layer F.Fab)
       (effects (font (size 0.4 0.4) (thickness 0.06)))
     )
@@
     (fp_line (start -0.8 -0.4) (end 0.8 -0.4) (layer F.Fab) (width 0.1))
     (fp_line (start -0.8 0.4) (end -0.8 -0.4) (layer F.Fab) (width 0.1))
-    (pad 2 smd roundrect (at 0.875 0) (size 1.05 0.95) (layers "L1_(Top)" F.Paste F.Mask) (roundrect_rratio 0.25)
+    (pad 2 smd roundrect (at 0.875 0 90) (size 1.05 0.95) (layers "L1_(Top)" F.Paste F.Mask) (roundrect_rratio 0.25)
       (net 243 /PHY.RMII0_RXD0\P0MODE0))
-    (pad 1 smd roundrect (at -0.875 0) (size 1.05 0.95) (layers "L1_(Top)" F.Paste F.Mask) (roundrect_rratio 0.25)
+    (pad 1 smd roundrect (at -0.875 0 90) (size 1.05 0.95) (layers "L1_(Top)" F.Paste F.Mask) (roundrect_rratio 0.25)
       (net 226 /RMII0_RXD0))
     (model ${KISYS3DMOD}/Resistor_SMD.3dshapes/R_0603_1608Metric.wrl
@@
   )
   (module Resistor_SMD:R_0603_1608Metric_Pad1.05x0.95mm_HandSolder (layer "L1_(Top)")
-    (at 89.35 37.28)
+    (at 144.55 73.8 90)
     (descr "Resistor SMD 0603 (1608 Metric), square (rectangular) end terminal, IPC_7351 nominal with elongated pad for handsoldering. (Body size source: http://www.tortai-tech.com/upload/download/2011102023233369053.pdf), generated with kicad-footprint-generator")
     (tags "resistor handsolder")
     (attr smd)
-    (fp_text reference R23 (at 0 -1.43) (layer F.SilkS)
+    (fp_text reference R23 (at 0 -1.43 90) (layer F.SilkS)
       (effects (font (size 1 1) (thickness 0.15)))
     )
-    (fp_text value 100 (at 0 1.43) (layer F.Fab)
+    (fp_text value 100 (at 0 1.43 90) (layer F.Fab)
       (effects (font (size 1 1) (thickness 0.15)))
     )
-    (fp_text user %R (at 0 0) (layer F.Fab)
+    (fp_text user %R (at 0 0 90) (layer F.Fab)
       (effects (font (size 0.4 0.4) (thickness 0.06)))
     )
@@
     (fp_line (start -0.8 -0.4) (end 0.8 -0.4) (layer F.Fab) (width 0.1))
     (fp_line (start -0.8 0.4) (end -0.8 -0.4) (layer F.Fab) (width 0.1))
-    (pad 2 smd roundrect (at 0.875 0) (size 1.05 0.95) (layers "L1_(Top)" F.Paste F.Mask) (roundrect_rratio 0.25)
+    (pad 2 smd roundrect (at 0.875 0 90) (size 1.05 0.95) (layers "L1_(Top)" F.Paste F.Mask) (roundrect_rratio 0.25)
       (net 242 /PHY.RMII0_RXD1\P0MODE1))
-    (pad 1 smd roundrect (at -0.875 0) (size 1.05 0.95) (layers "L1_(Top)" F.Paste F.Mask) (roundrect_rratio 0.25)
+    (pad 1 smd roundrect (at -0.875 0 90) (size 1.05 0.95) (layers "L1_(Top)" F.Paste F.Mask) (roundrect_rratio 0.25)
       (net 227 /RMII0_RXD1))
     (model ${KISYS3DMOD}/Resistor_SMD.3dshapes/R_0603_1608Metric.wrl
@@
   )
   (module Resistor_SMD:R_0603_1608Metric_Pad1.05x0.95mm_HandSolder (layer "L1_(Top)")
-    (at 125.05 36.1 180)
+    (at 146.25 73.8 90)
     (descr "Resistor SMD 0603 (1608 Metric), square (rectangular) end terminal, IPC_7351 nominal with elongated pad for handsoldering. (Body size source: http://www.tortai-tech.com/upload/download/2011102023233369053.pdf), generated with kicad-footprint-generator")
     (tags "resistor handsolder")
     (attr smd)
-    (fp_text reference R22 (at 0.1 -1.35) (layer F.SilkS)
+    (fp_text reference R22 (at 0.1 -1.35 90) (layer F.SilkS)
       (effects (font (size 1 1) (thickness 0.15)))
     )
-    (fp_text value 100 (at 0 1.43) (layer F.Fab)
+    (fp_text value 100 (at 0 1.43 90) (layer F.Fab)
       (effects (font (size 1 1) (thickness 0.15)))
     )
-    (fp_text user %R (at 0 0) (layer F.Fab)
+    (fp_text user %R (at 0 0 90) (layer F.Fab)
       (effects (font (size 0.4 0.4) (thickness 0.06)))
     )
@@
     (fp_line (start -0.8 -0.4) (end 0.8 -0.4) (layer F.Fab) (width 0.1))
     (fp_line (start -0.8 0.4) (end -0.8 -0.4) (layer F.Fab) (width 0.1))
-    (pad 2 smd roundrect (at 0.875 0 180) (size 1.05 0.95) (layers "L1_(Top)" F.Paste F.Mask) (roundrect_rratio 0.25)
+    (pad 2 smd roundrect (at 0.875 0 90) (size 1.05 0.95) (layers "L1_(Top)" F.Paste F.Mask) (roundrect_rratio 0.25)
       (net 241 /PHY.RMII0_CRSDV\P0MODE2))
-    (pad 1 smd roundrect (at -0.875 0 180) (size 1.05 0.95) (layers "L1_(Top)" F.Paste F.Mask) (roundrect_rratio 0.25)
+    (pad 1 smd roundrect (at -0.875 0 90) (size 1.05 0.95) (layers "L1_(Top)" F.Paste F.Mask) (roundrect_rratio 0.25)
       (net 228 /RMII0_CRSDV))
     (model ${KISYS3DMOD}/Resistor_SMD.3dshapes/R_0603_1608Metric.wrl
@@
   )
   (module Resistor_SMD:R_0603_1608Metric_Pad1.05x0.95mm_HandSolder (layer "L1_(Top)")
-    (at 125.1 38.9 180)
+    (at 147.95 73.8 90)
     (descr "Resistor SMD 0603 (1608 Metric), square (rectangular) end terminal, IPC_7351 nominal with elongated pad for handsoldering. (Body size source: http://www.tortai-tech.com/upload/download/2011102023233369053.pdf), generated with kicad-footprint-generator")
     (tags "resistor handsolder")
     (attr smd)
-    (fp_text reference R21 (at -0.1 -1.45) (layer F.SilkS)
+    (fp_text reference R21 (at -0.1 -1.45 90) (layer F.SilkS)
       (effects (font (size 1 1) (thickness 0.15)))
     )
-    (fp_text value 100 (at 0 1.43) (layer F.Fab)
+    (fp_text value 100 (at 0 1.43 90) (layer F.Fab)
       (effects (font (size 1 1) (thickness 0.15)))
     )
-    (fp_text user %R (at 0 0) (layer F.Fab)
+    (fp_text user %R (at 0 0 90) (layer F.Fab)
       (effects (font (size 0.4 0.4) (thickness 0.06)))
     )
@@
     (fp_line (start -0.8 -0.4) (end 0.8 -0.4) (layer F.Fab) (width 0.1))
     (fp_line (start -0.8 0.4) (end -0.8 -0.4) (layer F.Fab) (width 0.1))
-    (pad 2 smd roundrect (at 0.875 0 180) (size 1.05 0.95) (layers "L1_(Top)" F.Paste F.Mask) (roundrect_rratio 0.25)
+    (pad 2 smd roundrect (at 0.875 0 90) (size 1.05 0.95) (layers "L1_(Top)" F.Paste F.Mask) (roundrect_rratio 0.25)
       (net 240 /PHY.RMII0_RXERR\P0AD0))
-    (pad 1 smd roundrect (at -0.875 0 180) (size 1.05 0.95) (layers "L1_(Top)" F.Paste F.Mask) (roundrect_rratio 0.25)
+    (pad 1 smd roundrect (at -0.875 0 90) (size 1.05 0.95) (layers "L1_(Top)" F.Paste F.Mask) (roundrect_rratio 0.25)
       (net 229 /RMII0_RXERR))
     (model ${KISYS3DMOD}/Resistor_SMD.3dshapes/R_0603_1608Metric.wrl

Commit message: updating deprecated library footprints. Sch/pcb back in sync on new system
Parts:
- added C38: 10n, Capacitor_SMD:C_0603_1608Metric_Pad1.08x0.95mm_HandSolder, F.Cu at (185.4, 33.0)
- added C39: 10n, Capacitor_SMD:C_0603_1608Metric_Pad1.08x0.95mm_HandSolder, F.Cu at (194.1, 36.8)
- added C40: 10n, Capacitor_SMD:C_0603_1608Metric_Pad1.08x0.95mm_HandSolder, F.Cu at (187.1, 27.1)
- added C41: 0.1, Capacitor_SMD:C_1206_3216Metric_Pad1.33x1.80mm_HandSolder, F.Cu at (177.2, 24.1)
- added C42: 0.1, Capacitor_SMD:C_1206_3216Metric_Pad1.33x1.80mm_HandSolder, F.Cu at (177.2, 27.5)
- added C43: 1u, Capacitor_SMD:C_1206_3216Metric_Pad1.33x1.80mm_HandSolder, F.Cu at (183.2, 24.1)
- added C44: 1u, Capacitor_SMD:C_1206_3216Metric_Pad1.33x1.80mm_HandSolder, F.Cu at (177.2, 30.8)
- added C45: 10n, Capacitor_SMD:C_0603_1608Metric_Pad1.08x0.95mm_HandSolder, F.Cu at (181.1, 33.8)
- added C46: 470p, Capacitor_SMD:C_0603_1608Metric_Pad1.08x0.95mm_HandSolder, F.Cu at (193.2, 23.7)
- added C47: 470p, Capacitor_SMD:C_0603_1608Metric_Pad1.08x0.95mm_HandSolder, F.Cu at (176.3, 39.2)
- added C48: 10n, Capacitor_SMD:C_0603_1608Metric_Pad1.08x0.95mm_HandSolder, F.Cu at (187.1, 29.6)
- added C49: 10n, Capacitor_SMD:C_0603_1608Metric_Pad1.08x0.95mm_HandSolder, F.Cu at (191.5, 26.7)
- added C50: 10n, Capacitor_SMD:C_0603_1608Metric_Pad1.08x0.95mm_HandSolder, F.Cu at (181.1, 36.3)
- added C51: 10n, Capacitor_SMD:C_0603_1608Metric_Pad1.08x0.95mm_HandSolder, F.Cu at (176.3, 36.7)
- added C52: 22n, Capacitor_SMD:C_0805_2012Metric_Pad1.18x1.45mm_HandSolder, F.Cu at (188.6, 24.0)
- added C53: 22n, Capacitor_SMD:C_0805_2012Metric_Pad1.18x1.45mm_HandSolder, F.Cu at (182.6, 27.3)
- added FB2: Ferrite_Bead_Small, Inductor_SMD:L_1206_3216Metric_Pad1.42x1.75mm_HandSolder, F.Cu at (-116.9, -67.4)
- added R25: 10k, Resistor_SMD:R_0603_1608Metric_Pad0.98x0.95mm_HandSolder, F.Cu at (197.5, 23.7)
- added R54: 10k, Resistor_SMD:R_0603_1608Metric_Pad0.98x0.95mm_HandSolder, F.Cu at (185.4, 35.5)
- added R55: 10k, Resistor_SMD:R_0603_1608Metric_Pad0.98x0.95mm_HandSolder, F.Cu at (180.7, 38.8)
- added R56: 10k, Resistor_SMD:R_0603_1608Metric_Pad0.98x0.95mm_HandSolder, F.Cu at (191.5, 29.2)
- added R57: 10k, Resistor_SMD:R_0603_1608Metric_Pad0.98x0.95mm_HandSolder, F.Cu at (195.8, 26.2)
- added R58: 10k, Resistor_SMD:R_0603_1608Metric_Pad0.98x0.95mm_HandSolder, F.Cu at (180.7, 41.3)
- added R59: 10, Resistor_SMD:R_0603_1608Metric_Pad0.98x0.95mm_HandSolder, F.Cu at (189.8, 32.1)
- added R60: 10, Resistor_SMD:R_0603_1608Metric_Pad0.98x0.95mm_HandSolder, F.Cu at (185.4, 38.0)
- added R61: 1.5k, Resistor_SMD:R_0603_1608Metric_Pad0.98x0.95mm_HandSolder, F.Cu at (201.8, 23.7)
- added R62: 1.5k, Resistor_SMD:R_0603_1608Metric_Pad0.98x0.95mm_HandSolder, F.Cu at (198.5, 31.2)
- added R63: 10k, Resistor_SMD:R_0603_1608Metric_Pad0.98x0.95mm_HandSolder, F.Cu at (195.8, 28.7)
- added R64: 10k, Resistor_SMD:R_0603_1608Metric_Pad0.98x0.95mm_HandSolder, F.Cu at (200.2, 26.2)
- added R65: 10k, Resistor_SMD:R_0603_1608Metric_Pad0.98x0.95mm_HandSolder, F.Cu at (185.0, 40.5)
- added R66: 10k, Resistor_SMD:R_0603_1608Metric_Pad0.98x0.95mm_HandSolder, F.Cu at (194.1, 31.7)
- added R67: 33, Resistor_SMD:R_0603_1608Metric_Pad0.98x0.95mm_HandSolder, F.Cu at (189.8, 37.1)
- added R68: 33, Resistor_SMD:R_0603_1608Metric_Pad0.98x0.95mm_HandSolder, F.Cu at (206.2, 23.7)
- added R69: 10k, Resistor_SMD:R_0603_1608Metric_Pad0.98x0.95mm_HandSolder, F.Cu at (189.8, 39.6)
- added R70: 10k, Resistor_SMD:R_0603_1608Metric_Pad0.98x0.95mm_HandSolder, F.Cu at (194.1, 34.2)
- added R71: 0, Resistor_SMD:R_0805_2012Metric_Pad1.20x1.40mm_HandSolder, F.Cu at (176.5, 34.0)
- added R72: 0, Resistor_SMD:R_0805_2012Metric_Pad1.20x1.40mm_HandSolder, F.Cu at (182.5, 30.3)
- added R73: 33, Resistor_SMD:R_0603_1608Metric_Pad0.98x0.95mm_HandSolder, F.Cu at (200.2, 28.7)
- added R74: 33, Resistor_SMD:R_0603_1608Metric_Pad0.98x0.95mm_HandSolder, F.Cu at (204.5, 26.2)
- added R75: 12.1k, Resistor_SMD:R_0603_1608Metric_Pad0.98x0.95mm_HandSolder, F.Cu at (198.5, 41.3)
- added R76: 0, Resistor_SMD:R_0603_1608Metric_Pad0.98x0.95mm_HandSolder, F.Cu at (189.8, 34.6)
- added R77: 12.1k, Resistor_SMD:R_0603_1608Metric_Pad0.98x0.95mm_HandSolder, F.Cu at (198.5, 33.8)
- added R78: 0, Resistor_SMD:R_0603_1608Metric_Pad0.98x0.95mm_HandSolder, F.Cu at (194.1, 39.3)
- added R79: 49.9, Resistor_SMD:R_0603_1608Metric_Pad0.98x0.95mm_HandSolder, F.Cu at (202.8, 31.2)
- added R80: 49.9, Resistor_SMD:R_0603_1608Metric_Pad0.98x0.95mm_HandSolder, F.Cu at (204.5, 28.7)
- added R81: 49.9, Resistor_SMD:R_0603_1608Metric_Pad0.98x0.95mm_HandSolder, F.Cu at (198.5, 36.3)
- added R82: 49.9, Resistor_SMD:R_0603_1608Metric_Pad0.98x0.95mm_HandSolder, F.Cu at (202.8, 33.8)
- added R83: 49.9, Resistor_SMD:R_0603_1608Metric_Pad0.98x0.95mm_HandSolder, F.Cu at (198.5, 38.8)
- added R84: 49.9, Resistor_SMD:R_0603_1608Metric_Pad0.98x0.95mm_HandSolder, F.Cu at (207.2, 31.2)
- added R85: 49.9, Resistor_SMD:R_0603_1608Metric_Pad0.98x0.95mm_HandSolder, F.Cu at (202.8, 36.3)
- added R86: 49.9, Resistor_SMD:R_0603_1608Metric_Pad0.98x0.95mm_HandSolder, F.Cu at (207.2, 33.8)
- added TP3: TestPoint, TestPoint:TestPoint_Keystone_5019_Minature, F.Cu at (-117.0, -63.8)
- added TP4: TestPoint, TestPoint:TestPoint_Keystone_5019_Minature, F.Cu at (-111.1, -67.1)
- added X1: ASE-xxxMHz, Oscillator:Oscillator_SMD_Abracon_ASE-4Pin_3.2x2.5mm, F.Cu at (-111.6, -62.9)
- added X2: ASE-xxxMHz, Oscillator:Oscillator_SMD_Abracon_ASE-4Pin_3.2x2.5mm, F.Cu at (-105.7, -66.9)
- R21, R22, R23, R24, R26, R27: value 100 -> 10
Connections:
- net /PHY.RXCLK\P0AD1 renamed /PHY.RMII0_RXCLK\P0AD1
- net Net-(R30-Pad1) renamed /PHY.RMII1_RXERR\P1AD0
- net Net-(U1-Pad117) renamed /QSPI0_SS0
- net Net-(U1-Pad118) renamed /QSPI0_CLK
- net Net-(U1-Pad119) renamed /QSPI0_MOSI0
- net Net-(U1-Pad120) renamed /QSPI0_MISO0
- net Net-(U1-Pad121) renamed /QSPI0_MOSI1
- net Net-(U1-Pad122) renamed /QSPI0_MISO1
- net Net-(U1-Pad132) renamed /JTAG.TDO
- net Net-(U1-Pad133) renamed /JTAG.TCK
- net Net-(U1-Pad134) renamed /JTAG.TMS
- net Net-(U1-Pad135) renamed /JTAG.TDI
- net Net-(U1-Pad136) renamed /JTAG.TRST
- J4 pad 13: Net-(J4-Pad13) -> GND
- J4 pad R4: Net-(J4-PadR4) -> VDDA
- J4 pad R5: Net-(J4-PadR5) -> VDDA
- J4 pad R8: Net-(J4-PadR8) -> GND
- J5 pad 13: Net-(J5-Pad13) -> GND
- J5 pad R4: Net-(J5-PadR4) -> VDDA
- J5 pad R5: Net-(J5-PadR5) -> VDDA
- J5 pad R8: Net-(J5-PadR8) -> GND
- R26 pad 1: Net-(R26-Pad1) -> /RMII1_RXERR
- R26 pad 2: Net-(R26-Pad2) -> /PHY.RMII1_RXER\P1AD0
- R27 pad 1: Net-(R27-Pad1) -> /RMII1_CRSDV
- R27 pad 2: Net-(R27-Pad2) -> /PHY.RMII1_CRSDV\P1MODE2
- R34 pad 1: Net-(R34-Pad1) -> /PHY.RMII1_RXCLK\P1AD1
- R35 pad 1: Net-(R34-Pad1) -> /PHY.RMII1_RXCLK\P1AD1
- R38 pad 1: Net-(R38-Pad1) -> /P1AD2
- R39 pad 1: Net-(R38-Pad1) -> /P1AD2
- R42 pad 1: Net-(R42-Pad1) -> /PHY.RMII1_RXD0\P1MODE0
- R43 pad 1: Net-(R42-Pad1) -> /PHY.RMII1_RXD0\P1MODE0
- R44 pad 1: Net-(R44-Pad1) -> /PHY.RMII1_RXD1\P1MODE1
- R45 pad 1: Net-(R44-Pad1) -> /PHY.RMII1_RXD1\P1MODE1
- R48 pad 1: Net-(R48-Pad1) -> /PHY.RMII0_CRSDV\P0MODE2
- R49 pad 1: Net-(R48-Pad1) -> /PHY.RMII0_CRSDV\P0MODE2
- U1 pad 40: Net-(U1-Pad40) -> /FLASHCFG1
- U1 pad 41: Net-(U1-Pad41) -> /FLASHCFG0
- U1 pad 44: Net-(U1-Pad44) -> /UART_DBG_EN
- U1 pad 46: Net-(U1-Pad46) -> /WDT_DISABLE
- U1 pad 48: Net-(U1-Pad48) -> /BTSEL0
- U1 pad 49: Net-(U1-Pad49) -> /BTSEL1
- U2 pad 1: Net-(U2-Pad1) -> VDDA
- U2 pad 10: Net-(U2-Pad10) -> /PHY.RMII1_RXD1\P1MODE1
- U2 pad 11: Net-(U2-Pad11) -> /PHY.RMII1_RXD0\P1MODE0
- U2 pad 13: Net-(U2-Pad13) -> /PHY.RMII1_RXER\P1AD0
- U2 pad 15: Net-(U2-Pad15) -> /PHY.RMII1_CRSDV\P1MODE2
- U2 pad 16: Net-(U2-Pad16) -> /RMII1_MDIO
- U2 pad 17: Net-(U2-Pad17) -> /RMII1_MDC
- U2 pad 21: Net-(U2-Pad21) -> /RMII1_TXEN
- U2 pad 22: Net-(U2-Pad22) -> /RMII1_TXD0
- U2 pad 23: Net-(U2-Pad23) -> /RMII1_TXD1
- U2 pad 24: Net-(U2-Pad24) -> GND
- U2 pad 25: Net-(U2-Pad25) -> GND
- U2 pad 27: Net-(U2-Pad27) -> VDDA
- U2 pad 28: Net-(U2-Pad28) -> Net-(J5-PadR2)
- U2 pad 29: Net-(U2-Pad29) -> Net-(J5-PadR1)
- U2 pad 30: Net-(U2-Pad30) -> Net-(J5-PadR6)
- U2 pad 31: Net-(U2-Pad31) -> Net-(J5-PadR3)
- U2 pad 33: Net-(U2-Pad33) -> GND
- U2 pad 5: Net-(U2-Pad5) -> /P1_XTALI
- U2 pad 6: +1V2 -> /P1_CORE
- U2 pad 7: Net-(U2-Pad7) -> /PHY.RMII1_RXCLK\P1AD1
- U2 pad 8: Net-(U2-Pad8) -> /P1AD2
- U3 pad 1: Net-(U3-Pad1) -> VDDA
- U3 pad 19: Net-(U3-Pad19) -> /P0_nRST
- U3 pad 27: Net-(U3-Pad27) -> VDDA
- U3 pad 28: Net-(U3-Pad28) -> Net-(J4-PadR2)
- U3 pad 29: Net-(U3-Pad29) -> Net-(J4-PadR1)
- U3 pad 30: Net-(U3-Pad30) -> Net-(J4-PadR6)
- U3 pad 31: Net-(U3-Pad31) -> Net-(J4-PadR3)
- U3 pad 33: Net-(U3-Pad33) -> GND
- U3 pad 5: Net-(R25-Pad2) -> /P0_XTALI
- U3 pad 6: +1V2 -> /P0_CORE

Commit message: Some rough placement grouping and power routing
Parts:
- removed the R25 at (141.2, 73.8)
- C14, C19, C44, C47, FB1, R30, R31, R32, R33, R34, R35, R36, R37, R38, R39, R40, R41, R42, R43, R44, R45, R46, R47, R48, R49, R50, R51, R52, R53, R71: moved to B.Cu
- moved X1 383.8 mm to (262.2, 23.8)
- moved X2 379.2 mm to (263.9, 18.2)
- moved FB2 379.2 mm to (252.7, 17.7)
- moved TP3 379.2 mm to (252.6, 21.3)
- moved TP4 379.2 mm to (258.5, 18.0)
- moved C29 154.7 mm to (123.2, 63.2)
- moved C27 150.1 mm to (119.3, 68.4), turned to 90 degrees
- moved C14 145.5 mm to (134.0, 71.4), turned to 90 degrees
- moved Y1 134.2 mm to (134.6, 109.0), turned to 180 degrees
- moved C28 127.8 mm to (125.9, 67.4), turned to 270 degrees
- moved U4 125.5 mm to (122.4, 68.1), turned to 90 degrees
- moved R2 122.1 mm to (148.5, 71.9), turned to 180 degrees
- moved U6 121.3 mm to (115.2, 76.7)
- moved R8 119.5 mm to (119.8, 80.3), turned to 180 degrees
- moved R9 118.8 mm to (118.5, 74.7), turned to 90 degrees
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Connections:
- R30 pad 1: /PHY.RMII1_RXERR\P1AD0 -> /PHY.RMII1_RXER\P1AD0
- R31 pad 1: /PHY.RMII1_RXERR\P1AD0 -> /PHY.RMII1_RXER\P1AD0
- R48 pad 1: /PHY.RMII0_CRSDV\P0MODE2 -> /PHY.RMII1_CRSDV\P1MODE2
- R49 pad 1: /PHY.RMII0_CRSDV\P0MODE2 -> /PHY.RMII1_CRSDV\P1MODE2
Routing:
- net +3V3: track 16.7 -> 143.6 mm, vias 0 -> 15
- net +1V2: track 0.00 -> 85.9 mm, vias 0 -> 10
- net GND: track 0.00 -> 53.5 mm, vias 0 -> 38
- net +3.3VA: track 0.00 -> 11.3 mm, vias 0 -> 2
- net /1V8_EN: track 0.00 -> 10.7 mm
- net /PHY.RMII0_RXCLK\P0AD1: track 0.00 -> 10.1 mm, vias 0 -> 1
- net Net-(R6-Pad2): track 0.00 -> 9.66 mm
- net /PHY.RMII0_RXD1\P0MODE1: track 0.00 -> 6.88 mm, vias 0 -> 1
- net /FLASHCFG1: track 0.00 -> 6.83 mm
- net /BTSEL1: track 0.00 -> 6.58 mm
- net /FLASHCFG0: track 0.00 -> 6.40 mm
- net /UART_DBG_EN: track 0.00 -> 6.33 mm
- net /P0AD2: track 0.00 -> 6.20 mm, vias 0 -> 1
- net /BTSEL0: track 0.00 -> 6.18 mm
- net +1V8: track 0.00 -> 6.18 mm, vias 0 -> 2
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- added copper zone on B.Cu, net +1V2
- added copper zone on B.Cu, net +3V3
